File: Personal Audio Recorder/Board.sch (EAGLE design)
At the start: 49 parts, among them IC1 MCP1703CB, IC2 MCP73831/OT, J1 PIC_ICSP_MINI_5_PIN, J2 503182-1852, J4 1050170001, U1 XC6204B332MR-SOT23-5

Commit message: Redid board
Parts:
- removed C5: .1uF, rcl:C-USC0603
- removed IC1: MCP1703CB, linear:MCP1703CB
- removed IC2: MCP73831/OT, adafruit:MCP73831/OT
- removed J4: 1050170001, 1050170001:1050170001
- removed PAD1, PAD2: (no value), wirepad:SMD2
- removed Q1: (no value), Extras:ELECTRET
- removed R16, R17: 470, rcl:R-US_R0603
- removed TP1, TP2, TP3: TPTP10R, BeagleBone_Blue_R3:TPTP10R
- removed U$1: SIT1532AC-J5-DCC, Extras:SIT1532AC-J5-DCC
- removed U$2: PIC32MX274F256B, Extras:PIC32MX274F256B
- removed VR1: TC33X-2-104E (100K), microbuilder:TRIMPOTTC33X-2
- added BAT+, BAT-: (no value), wirepad:SMD2
- added C11: 10uF, resistor:C-USC0603
- added CON1: 1050170001, 1050170001:1050170001
- added MIC: (no value), Extras:ELECTRET
- added SJ1: (no value), Extras:SJ2WJUMPER
- added U2: MCP73831/OT, adafruit:MCP73831/OT
- added U3: MCP1703CB, linear:MCP1703CB
- added U4: MAX9814TDFN14, adafruit:MAX9814TDFN14
- added X1: SIT1532AC-J5-DCC, Extras:SIT1532AC-J5-DCC
- C1: value 100pF -> 0.1uF; device rcl:C-USC0603 -> resistor:C-USC0603
- C10: value .1uF -> .01uF; device rcl:C-USC0603 -> resistor:C-USC0603
- C2: value 10pF -> 2.2uF; device rcl:C-USC0603 -> resistor:C-USC0603
- C3: value 100pF -> 0.47uF; device rcl:C-USC0603 -> resistor:C-USC0603
- C4: value 1uF -> 0.1uF; device rcl:C-USC0603 -> resistor:C-USC0603
- C6, C7: value .1uF -> 0.1uF; device rcl:C-USC0603 -> resistor:C-USC0603
- C8, C9: device rcl:C-USC0603 -> resistor:C-USC0603
- R1, R2: value 1M -> 10K; device rcl:R-US_R0603 -> resistor:R-US_R0603
- R10, R11, R12, R13, R14, R6, R7, R8, R9: device rcl:R-US_R0603 -> resistor:R-US_R0603
- R15, R4: value 1K -> 470; device rcl:R-US_R0603 -> resistor:R-US_R0603
- R3: value 1K -> 10K; device rcl:R-US_R0603 -> resistor:R-US_R0603
- R5: value 10K -> 100; device rcl:R-US_R0603 -> resistor:R-US_R0603
- U1: value XC6204B332MR-SOT23-5 -> PIC32MX274F256B; device Extras:MAX4466 -> Extras:PIC32MX274F256B
- renumbered J1 to CON2
Connections:
- removed net LED3: LED3.A, U$2.RB3
- removed net N$14: CON2.PGD, U$2.RB0
- removed net N$15: CON2.PGC, U$2.RB1
- new net D+: CON1.3, U1.D+
- new net D-: CON1.2, U1.D-
- new net LED1: LED2.A, U1.RB0
- new net N$16: C3.1, U4.BIAS
- new net N$22: L2.2, R5.2
- new net N$23: SJ1.2, U4.GAIN
- new net PGC: CON2.PGC, U1.RA1
- new net PGD: CON2.PGD, U1.RA0
- new net VCAP: C11.1, U1.VCAP
- net AVCC: now also SJ1.1, U1.AVDD, U4./SHDN, U4.VDD; no longer R1.2, R3.2, U$2.AVDD, U1.VCC
- net GND: now also BAT-.P, C11.2, C2.2, C3.2, CON1.5, CON1.SHIELD, MIC.1, R1.2, R11.1, R14.1, R6.1, SJ1.3, U$3.P$1, U$3.P$2, U$3.P$3, U1.AVSS, U1.VSS@1, U1.VSS@2, U1.VSS@3, U2.VSS, U3.GND, U4.A/R, U4.EP, U4.GND, U4.NC1, U4.NC2, X1.GND@1, X1.GND@2; no longer C4.2, C5.2, IC1.GND, IC2.VSS, J4.5, J4.SHIELD, PAD2.P, Q1.1, R11.2, R16.1, R17.1, R2.1, TP2.TP, U$1.GND@1, U$1.GND@2, U$2.AVSS, U$2.VSS@1, U$2.VSS@2, U$2.VSS@3, U1.GND
- net LED2: now also LED3.A, U1.RB1; no longer LED2.A, U$2.RB2
- net MICOUT: now also U1.RB2, U4.MICOUT; no longer C3.2, TP3.TP, U$2.RB13, U1.OUT, VR1.A, VR1.S
- net MISO: now also R7.1, U1.RB5; no longer R7.2, U$2.RB5
- net MMC_SS: now also R11.2, U1.RB8; no longer R11.1, U$2.RB8
- net MOSI: now also R8.1, U1.RB13; no longer R10.2, U$2.RA4
- net N$1: now also U4.CT; no longer R3.1, R4.2
- net N$10: now also R4.1, U2.STAT; no longer IC2.STAT, R14.1
- net N$11: now also R12.2; no longer R12.1
- net N$12: now also R6.2, U2.PROG; no longer IC2.PROG, R15.2
- net N$13: now also U1.!MCLR; no longer U$2.!MCLR
- net N$17: now also BAT+.P, U2.VBAT, U3.VI; no longer IC1.VI, IC2.VBAT, PAD1.P
- net N$18: now also R14.2; no longer R16.2
- net N$19: now also R15.2; no longer R17.2
- net N$2: now also U4.CG; no longer Q1.2, R4.1
- net N$21: now also C4.1, U4.MICIN; no longer R5.2, VR1.E
- net N$3: now also R3.1, U4.MICBIAS; no longer C2.2, R1.1, U1.IN+
- net N$4: now also CON1.1, U2.VDD; no longer IC2.VDD, J4.1
- net N$5: now also R10.1; no longer R9.2
- net N$6: now also R1.1, R2.1, U4.TH; no longer C3.1, R5.1, R6.2, U1.IN-
- net N$7: now also R9.1; no longer R8.2
- net N$8: now also C4.2, MIC.2, R3.2; no longer C4.1, R6.1
- net N$9: now also R4.2; no longer R14.2
- net PB: now also U1.RB7; no longer U$2.RB7
- net RTCCCLK: now also U1.RB4, X1.CLKOUT; no longer U$1.CLKOUT, U$2.RB4
- net SCK: now also U1.RB14; no longer U$2.RB14
- net VCC: now also R10.2, R12.1, R5.1, R7.2, R8.2, R9.2, U1.VDD@1, U1.VUSB3V3, U3.VO, X1.VDD; no longer C5.1, IC1.VO, L2.2, R10.1, R12.2, R7.1, R8.1, R9.1, TP1.TP, U$1.VDD, U$2.VDD@1, U$2.VUSB3V3
Other:
- moved on the sheet: C1, C10, C2, C3, C4, C8, C8/TANT, C9, J2, L1, L2, R1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

Commit message: Rev 1.2 board done and sent off
Parts:
- added R16, R17: 00, resistor:R-US_R0603
- R1: value 10K -> 100k
- R2: value 10K -> 150K
- R3: value 10K -> 2.2K
Connections:
- new net N$14: U1.RA2
- new net SD_SW: J2.SWITCH, U1.RA4
- new net USBID: CON1.4, U1.RB5
- new net VBUS: C8.1, CON1.1, LED1.A, U1.VBUS, U2.VDD
- net AVCC: now also R16.2
- net GND: now also R17.2; no longer U4.A/R
- net MISO: now also U1.RB8; no longer U1.RB5
- net MMC_SS: now also U1.RB9; no longer U1.RB8
- net N$4: now also R16.1, R17.1, U4.A/R; no longer C8.1, CON1.1, LED1.A, U2.VDD
